File: sbc/kicad/sheet1.sch (KiCad schematic (older format))
At the start: 32 parts, among them J1 POWER, J2 5V POWER, U1 LM7805, U25 74LS00, U4 74LS04

Commit message: Updates, start of PCB.
Parts:
- removed D3: 1N4001 X4, symbol Device:D_Bridge_+-AA
- added D2, D3, D5, D6: 1N4001, Diode_THT:D_DO-41_SOD81_P10.16mm_Horizontal, symbol Diode:1N4001
- C1, C10, C11, C12, C13, C14, C15, C16, C17, C18, C19, C20, C21, C3, C4, C5, C6, C7, C8, C9: footprint (none) -> Capacitor_THT:C_Disc_D4.3mm_W1.9mm_P5.00mm
- C2: footprint (none) -> Capacitor_THT:CP_Radial_D5.0mm_P2.00mm
- D7: renamed from D4; footprint (none) -> LED_THT:LED_D2.0mm_W4.8mm_H2.5mm_FlatTop
- J1, J2: footprint (none) -> Connector_PinHeader_2.54mm:PinHeader_1x02_P2.54mm_Vertical
- R1, R2: footprint (none) -> Resistor_THT:R_Axial_DIN0204_L3.6mm_D1.6mm_P7.62mm_Horizontal
- U2: renamed from U25; footprint (none) -> Package_DIP:DIP-14_W7.62mm_Socket
- U3: renamed from U4; footprint (none) -> Package_DIP:DIP-14_W7.62mm_Socket
- renumbered D2 to D4
Connections:
- net GND: now also D2.2 (A), D5.2 (A)
- net at C1.1, J1.1 (In), R1.2: now also D2.1 (K), D3.2 (A)
- net at C4.1, J1.2 (Ext): now also D5.1 (K), D6.2 (A)
- net at C2.1, U1.1 (VI): now also D3.1 (K), D6.1 (K)
Other:
- moved on the sheet: C1, C4, J1
