File: sbc/kicad/sheet5.sch (KiCad schematic (older format))
At the start: 11 parts, among them J5 LTC, J6 EXPANSION, J7 PARALLEL PORT, J8 FTDI SERIAL, J9 USB POWER, U22 ATF16V8B, U23 74LS244, U24 74LS42, U25 74LS00, U4 74LS04

Commit message: Circuit updates.
Parts:
- removed J7: PARALLEL PORT, symbol Connector_Generic:Conn_02x10_Counter_Clockwise
- added J10: BAUD RATE, symbol Connector_Generic:Conn_02x06_Odd_Even
- added J3: Parallel Port, symbol Connector_Generic:Conn_02x12_Counter_Clockwise
- added J4: TX DATA SELECT, symbol Connector:Conn_01x03_Male
- added J7: RX DATA SELECT, symbol Connector:Conn_01x03_Male
- added RN9: 3K, Resistor_THT:R_Array_SIP9, symbol Device:R_Network08
Connections:
- net CA1: now also J3.9 (Pin_9)
- net CA2: now also J3.10 (Pin_10)
- net CB1: now also J3.16 (Pin_16)
- net CB2: now also J3.15 (Pin_15)
- net GND: now also J10.10 (Pin_10), J10.12 (Pin_12), J10.2 (Pin_2), J10.4 (Pin_4), J10.6 (Pin_6), J10.8 (Pin_8), J3.11 (Pin_11), J3.14 (Pin_14)
- net PA0: now also J3.1 (Pin_1), J4.3 (Pin_3)
- net PA1: now also J10.1 (Pin_1), J10.11 (Pin_11), J3.2 (Pin_2), RN9.2 (R1), RN9.7 (R6)
- net PA2: now also J10.3 (Pin_3), J3.3 (Pin_3), RN9.3 (R2)
- net PA3: now also J10.5 (Pin_5), J3.4 (Pin_4), RN9.4 (R3)
- net PA4: now also J10.7 (Pin_7), J3.5 (Pin_5), RN9.5 (R4)
- net PA5: now also J10.9 (Pin_9), J3.6 (Pin_6), RN9.6 (R5)
- net PA6: now also J3.7 (Pin_7)
- net PA7: now also J3.8 (Pin_8), J7.1 (Pin_1)
- net PB0: now also J3.24 (Pin_24)
- net PB1: now also J3.23 (Pin_23)
- net PB2: now also J3.22 (Pin_22)
- net PB3: now also J3.21 (Pin_21)
- net PB4: now also J3.20 (Pin_20)
- net PB5: now also J3.19 (Pin_19)
- net PB6: now also J3.18 (Pin_18)
- net PB7: now also J3.17 (Pin_17)
- net RXDATA: now also J7.3 (Pin_3); no longer J8.4 (Pin_4)
- net TXDATA: now also J4.1 (Pin_1); no longer J8.5 (Pin_5)
- net VCC: now also J9.2 (Pin_2), J3.12 (Pin_12), J3.13 (Pin_13), RN9.1 (common); no longer J9.1 (Pin_1)
- net at J8.3 (Pin_3): now also J9.1 (Pin_1); no longer J9.2 (Pin_2)
- new net: J7.2 (Pin_2), J8.4 (Pin_4)
- new net: J4.2 (Pin_2), J8.5 (Pin_5)
- no-connect marks 20 -> 22
Other:
- moved on the sheet: J8, J9, RN2, U22, U24

Commit message: Updates, start of PCB.
Parts:
- J10: footprint (none) -> Connector_PinHeader_2.54mm:PinHeader_2x06_P2.54mm_Vertical
- J3: renamed from J6; footprint (none) -> Connector_PinHeader_2.54mm:PinHeader_2x20_P2.54mm_Vertical
- J4: renamed from J5; footprint (none) -> Connector_PinHeader_2.54mm:PinHeader_1x03_P2.54mm_Vertical
- J5: renamed from J3; footprint (none) -> Connector_PinHeader_2.54mm:PinHeader_2x12_P2.54mm_Vertical
- J6: renamed from J4; footprint (none) -> Connector_PinHeader_2.54mm:PinHeader_1x03_P2.54mm_Vertical
- J7: footprint (none) -> Connector_PinHeader_2.54mm:PinHeader_1x03_P2.54mm_Vertical
- J8: renamed from J9; footprint (none) -> Connector_PinHeader_2.54mm:PinHeader_1x02_P2.54mm_Vertical
- J9: renamed from J8; footprint (none) -> Connector_PinHeader_2.54mm:PinHeader_1x06_P2.54mm_Vertical
- U2: renamed from U25; footprint (none) -> Package_DIP:DIP-14_W7.62mm_Socket
- U22, U23: footprint (none) -> Package_DIP:DIP-20_W7.62mm_Socket
- U24: footprint (none) -> Package_DIP:DIP-16_W7.62mm_Socket
- U3: renamed from U4; footprint (none) -> Package_DIP:DIP-14_W7.62mm_Socket
- renumbered RN2 to RN8
