File: sbc/kicad/6800sbc.kicad_pcb (KiCad board)
At the start: 2 copper layers, 188 x 193 mm, 164 parts, among them J1 AC/DC IN, J10 PA1, J11 SEGMENT TEST, J12 REG. POWER, J13 PA2, J14 PA3, J15 PA4, J16 PA5, J17 PA6, J2 5V IN, J3 EXPANSION, J4 LTC, J5 PARALLEL PORT, J6 TX DATA SELECT, J7 RX DATA SELECT, J8 USB POWER, J9 FTDI SERIAL, SW10 "9", SW11 "4", SW12 "5", SW13 "6", SW14 "1", SW15 "2", SW16 "3", SW17 "0", SW18 "RESET", SW2 "D", SW3 "E", SW4 "F", SW5 "A", SW6 "B", SW7 "C", SW8 "7", SW9 "8", U1 LM7805, U10 MAN71A, U11 MAN71A, U12 74LS259, U13 74LS259, U14 74LS259, U15 74LS259, U16 74LS259, U17 74LS259, U18 74LS244, U19 62256, U2 74LS00, U20 27128, U21 MC6802, U22 ATF16V8B, U23 74LS244, U24 74LS42, U3 74LS04, U4 6821, U5 MC6850, U6 MAN71A, U7 MAN71A, U8 MAN71A, U9 MAN71A, Y1 1.8432 MHz, Y2 3.579545 MHz

Commit message: Update PCB elayout and Gerber files for rev 1.0PCB.
Parts:
- Y2: value 3.579545 MHz -> 4 MHz
Connections:
- SW10 pad 2: Net-(SW10-Pad2) -> Net-(R58-Pad2)
- SW11 pad 2: Net-(SW11-Pad2) -> Net-(R57-Pad2)
- SW12 pad 2: Net-(SW11-Pad2) -> Net-(R57-Pad2)
- SW13 pad 2: Net-(SW11-Pad2) -> Net-(R57-Pad2)
- SW14 pad 2: Net-(SW14-Pad2) -> Net-(R56-Pad2)
- SW15 pad 2: Net-(SW14-Pad2) -> Net-(R56-Pad2)
- SW16 pad 2: Net-(SW14-Pad2) -> Net-(R56-Pad2)
- SW5 pad 2: Net-(SW5-Pad2) -> Net-(R59-Pad2)
- SW6 pad 2: Net-(SW5-Pad2) -> Net-(R59-Pad2)
- SW7 pad 2: Net-(SW5-Pad2) -> Net-(R59-Pad2)
- SW8 pad 2: Net-(SW10-Pad2) -> Net-(R58-Pad2)
- SW9 pad 2: Net-(SW10-Pad2) -> Net-(R58-Pad2)
Routing:
- net Net-(R56-Pad2): track 79.1 -> 149.7 mm
- net Net-(R57-Pad2): track 90.8 -> 154.4 mm
- net Net-(R58-Pad2): track 77.9 -> 138.1 mm
- net Net-(R59-Pad2): track 95.2 -> 152.8 mm
- net Net-(SW5-Pad2): track 42.1 -> 0.00 mm
- net Net-(SW14-Pad2): track 42.1 -> 0.00 mm
- net Net-(SW11-Pad2): track 42.1 -> 0.00 mm
- net Net-(SW10-Pad2): track 42.1 -> 0.00 mm

Commit message: Change C2 to 100uF.
Parts:
- C2: value 1000uF -> 100uF
Changed lines of the file:
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@@
       (effects (font (size 1 1) (thickness 0.15)))
     )
-    (fp_text value 1000uF (at 1 3.75) (layer F.Fab)
+    (fp_text value 100uF (at 1 3.75) (layer F.Fab)
       (effects (font (size 1 1) (thickness 0.15)))
     )
